File: KiCad project/user_interface.kicad_sch (KiCad schematic)
At the start: 11 parts, among them J4 B4B-XH-AM, J6 Conn_01x05, Q2 BC817, Q3 BC817, SW1 1101NE, SW2 1101NE

Commit message: Add HX711 scale controller schematic and clean up legacy components
- Add HX711_LoadCell_Summing child sheet with 4x MTMM-103-03-T-S-150 load cell connectors, summing resistors, and decoupling caps
- Add OLED_Header child sheet (4-pin I2C socket for SSD1306)
- Remove battery charger (MCP73871), LiPo connector, mic preamp, BME280, SD card from schematic
- Reconnect power path: +5V_USB -> FB1 -> +5V -> LDO
- Add Samtec MTMM-103-03-T-S-150 footprint library to fp-lib-table
- Assign footprints to HX711 passives (C12-C17, R15/R16) and net ties (NT1-NT3)
- Update PCB from schematic: add new scale components, remove legacy footprints
- Track fp-lib-table in git (uses portable ${KIPRJMOD} paths)

Co-Authored-By: Claude Sonnet 4.6 <noreply@anthropic.com>
Parts:
- removed J4: B4B-XH-AM, Footprints:JST_B4B-XH-AM__LF__SN_, symbol B4B-XH-AM__LF__SN_:B4B-XH-AM__LF__SN_
Other:
- note removed: "OLED display connector (I2C)"
- title: (none) -> ESP32 sensor board

Commit message: Schematic: native USB-Serial/JTAG replaces the CP2102N; strapping and I2C pull-ups; status LED
Review findings F1-F5 (docs/schematic-review-2026-09-18.md), Level 1 + 2:
- Removed U4 CP2102N and its support parts (R11, R12, R13, C9, C10, C11,
  D6, R18) and the DTR/RTS auto-program circuit (Q2, Q3, R33, R34).
  The QFN20 CP2102N has no DTR, so that circuit could never work.
- USB D+/D- now run from the ESD diode U5 to the module's native USB pins
  (IO19 = USB_D+, IO18 = USB_D-). Reset and download-mode entry are handled
  by the USB-Serial/JTAG peripheral.
- Pull-ups: R3 10k GPIO8 (required high for download boot), R4 10k GPIO2
  (recommended), R5 10k GPIO9/BOOT, R6/R7 4.7k SDA/SCL.
- D5 (green) + R14 kept as a status LED on GPIO7 (active-low).
- J6 expansion header re-pinned: 3.3V, GPIO10, U0TXD, U0RXD, GND.
- PWR_FLAG on GND moved to U5 (the one on the CP2102N ground went with it).
- firmware: logger on USB_SERIAL_JTAG, status_led on GPIO7, pin map notes.

ERC: 0 errors. Netlist connectivity checked pin-by-pin against the
intended design. Board not yet updated: run Update PCB from Schematic.

Co-Authored-By: Claude Fable 5.1 <noreply@anthropic.com>
Parts:
- removed Q2, Q3: BC817, Package_TO_SOT_SMD:SOT-23, symbol Transistor_BJT:BC817
- removed R33, R34: 10K, Resistor_SMD:R_0805_2012Metric, symbol Device:R
Connections:
- net GPIO18 renamed U0TXD
- net GPIO19 renamed U0RXD
- net GPIO8 renamed GPIO10

Commit message: Schematic: refresh sheet captions after the USB rework; drop the stale auto-program table
Co-Authored-By: Claude Fable 5.1 <noreply@anthropic.com>
Connections:
- net GND: no longer J6.5 (Pin_5)
Changed lines of the file:
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@@
-		)
-	)
-	(text_box "To learn more about the boot mode selection,\nsee documentation at https://txplo.re/esp32boot"
-		(exclude_from_sim no)
-		(at 198.755 131.445 0)
-		(size 29.845 11.43)
-		(margins 0.9525 0.9525 0.9525 0.9525)
-		(stroke
-			(width 0)
-			(type default)
-		)
-		(fill
-			(type none)
-		)
-		(effects
-			(font
-				(size 1.27 1.27)
-			)
-			(justify left top)
 		)
 	)
@@
 					(unit 1)
 				)
-			)
-		)
-	)
-	(symbol
-		(lib_id "power:GND")
-		(at 66.04 132.08 0)
-		(unit 1)
-		(exclude_from_sim no)
-		(in_bom yes)
-		(on_board yes)
-		(dnp no)
-		(fields_autoplaced yes)
-		(property "Reference" "#PWR058"
-			(at 66.04 138.43 0)
-			(effects
-				(font
-					(size 1.27 1.27)
-				)
-				(hide yes)
-			)
-		)
-		(property "Value" "GND"
-			(at 66.04 137.16 0)
-			(effects
-				(font
-					(size 1.27 1.27)
-				)
-			)
-		)
-		(property "Footprint" ""
-			(at 66.04 132.08 0)
-			(effects
-				(font
-					(size 1.27 1.27)
-				)
-				(hide yes)
-			)
-		)
-		(property "Datasheet" ""
-			(at 66.04 132.08 0)
-			(effects
-				(font
-					(size 1.27 1.27)
-				)
-				(hide yes)
-			)
-		)
-		(property "Description" "Power symbol creates a global label with name \"GND\" , ground"
-			(at 66.04 132.08 0)
-			(effects
-				(font
-					(size 1.27 1.27)
-				)
-				(hide yes)
-			)
-		)
-		(pin "1"
-		)
-		(instances
-			(project "ScaleController_RevA"
-				(path "/16c571a0-8550-4f05-972c-22b0701cbf02/09ec4a32-ddff-43cd-8e21-9ef822101853/9638f799-907f-4116-a2c8-fb3f1731f620"
-					(reference "#PWR058")
-					(unit 1)
-				)

Commit message: Fix: restore J6 ground symbol removed by mistake with the stale auto-program note
Co-Authored-By: Claude Fable 5.1 <noreply@anthropic.com>
Connections:
- net GND: now also J6.5 (Pin_5)
Changed lines of the file:
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@@
+		)
+	)
+	(symbol
+		(lib_id "power:GND")
+		(at 66.04 132.08 0)
+		(unit 1)
+		(exclude_from_sim no)
+		(in_bom yes)
+		(on_board yes)
+		(dnp no)
+		(fields_autoplaced yes)
+		(property "Reference" "#PWR058"
+			(at 66.04 138.43 0)
+			(effects
+				(font
+					(size 1.27 1.27)
+				)
+				(hide yes)
+			)
+		)
+		(property "Value" "GND"
+			(at 66.04 137.16 0)
+			(effects
+				(font
+					(size 1.27 1.27)
+				)
+			)
+		)
+		(property "Footprint" ""
+			(at 66.04 132.08 0)
+			(effects
+				(font
+					(size 1.27 1.27)
+				)
+				(hide yes)
+			)
+		)
+		(property "Datasheet" ""
+			(at 66.04 132.08 0)
+			(effects
+				(font
+					(size 1.27 1.27)
+				)
+				(hide yes)
+			)
+		)
+		(property "Description" "Power symbol creates a global label with name \"GND\" , ground"
+			(at 66.04 132.08 0)
+			(effects
+				(font
+					(size 1.27 1.27)
+				)
+				(hide yes)
+			)
+		)
+		(pin "1"
+		)
+		(instances
+			(project "ScaleController_RevA"
+				(path "/16c571a0-8550-4f05-972c-22b0701cbf02/09ec4a32-ddff-43cd-8e21-9ef822101853/9638f799-907f-4116-a2c8-fb3f1731f620"
+					(reference "#PWR058")
+					(unit 1)
+				)
+			)
 		)
 	)
