File: KiCad project/user_interface.kicad_sch (KiCad schematic)
At the start: 6 parts, among them J6 Conn_01x05, SW1 1101NE, SW2 1101NE

Commit message: Schematic: title blocks (Scale Controller, rev A, 2026-09-18, per-sheet comments); replace stale CP2102 and ESP32-S3 notes
Co-Authored-By: Claude Fable 5.1 <noreply@anthropic.com>
Other:
- company: (none) -> Steve Maegley
- title: ESP32 sensor board -> Scale Controller
Changed lines of the file:
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@@
 	(paper "A4")
 	(title_block
-		(title "ESP32 sensor board")
-		(rev "1")
-		(comment 1 "OLED Header")
+		(title "Scale Controller")
+		(date "2026-09-18")
+		(rev "A")
+		(company "Steve Maegley")
+		(comment 1 "Reset / boot buttons, expansion header J6")
 	)
 	(rectangle
