File: KiCad project/HX711_LoadCell_Summing.kicad_sch (KiCad schematic)
At the start: 16 parts, among them J3 MTMM-103-03-T-S-150, J5 MTMM-103-03-T-S-150, J7 MTMM-103-03-T-S-150, J8 MTMM-103-03-T-S-150, U6 HX711

Commit message: Unify 3.3V power nets; update PCB netlist
The HX711 sheet used power:+3.3V (4 symbols) and the OLED header sheet
used power:+3V3, which are separate nets from the SparkFun 3.3V symbol
used on the root, ESP32-C3 and UI sheets. The HX711 (VSUP/AVDD/DVDD,
decoupling, E+ net tie) and the OLED VCC pin were therefore unpowered.
Changed the five symbols' Value to 3.3V so they join the LDO rail:
one 3.3V net with 25 pins. ERC: 0 errors (87 library warnings, as before).

Updated PCB from schematic: +3.3V/+3V3 nets gone, 66 nets, 138 unrouted
connections (was 136). KiCad also normalized symbol-instance project
names in all sheets from the old KLP-5e parent names.

Co-Authored-By: Claude Fable 5.1 <noreply@anthropic.com>
Connections:
- net +3.3V renamed 3.3V
Changed lines of the file:
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@@
 		)
 		(instances
-			(project ""
+			(project "ScaleController_RevA"
 				(path "/16c571a0-8550-4f05-972c-22b0701cbf02/1a7f1cfb-b266-4842-99c6-585192ff3edb"
 					(reference "NT2")
@@
 		)
 		(instances
-			(project ""
+			(project "ScaleController_RevA"
 				(path "/16c571a0-8550-4f05-972c-22b0701cbf02/1a7f1cfb-b266-4842-99c6-585192ff3edb"
 					(reference "C15")
@@
 		)
 		(instances
-			(project ""
+			(project "ScaleController_RevA"
 				(path "/16c571a0-8550-4f05-972c-22b0701cbf02/1a7f1cfb-b266-4842-99c6-585192ff3edb"
 					(reference "U6")
@@
 		)
 		(instances
-			(project ""
+			(project "ScaleController_RevA"
 				(path "/16c571a0-8550-4f05-972c-22b0701cbf02/1a7f1cfb-b266-4842-99c6-585192ff3edb"
 					(reference "J5")
@@
 		)
 		(instances
-			(project ""
+			(project "ScaleController_RevA"
 				(path "/16c571a0-8550-4f05-972c-22b0701cbf02/1a7f1cfb-b266-4842-99c6-585192ff3edb"
 					(reference "R15")
@@
 		)
 		(instances
-			(project ""
+			(project "ScaleController_RevA"
 				(path "/16c571a0-8550-4f05-972c-22b0701cbf02/1a7f1cfb-b266-4842-99c6-585192ff3edb"
 					(reference "C13")
@@
 		)
 		(instances
-			(project ""
+			(project "ScaleController_RevA"
 				(path "/16c571a0-8550-4f05-972c-22b0701cbf02/1a7f1cfb-b266-4842-99c6-585192ff3edb"
 					(reference "J3")
@@
 			)
 		)
-		(property "Value" "+3.3V"
+		(property "Value" "3.3V"
 			(at 87.376 44.958 0)
 			(effects
@@
 		)
 		(instances
-			(project ""
+			(project "ScaleController_RevA"
 				(path "/16c571a0-8550-4f05-972c-22b0701cbf02/1a7f1cfb-b266-4842-99c6-585192ff3edb"
 					(reference "#PWR025")
@@
 			)
 		)
-		(property "Value" "+3.3V"
+		(property "Value" "3.3V"
 			(at 92.71 46.99 0)
 			(effects
@@
 		)
 		(instances
-			(project ""
+			(project "ScaleController_RevA"
 				(path "/16c571a0-8550-4f05-972c-22b0701cbf02/1a7f1cfb-b266-4842-99c6-585192ff3edb"
 					(reference "#PWR028")
@@
 		)
 		(instances
-			(project ""
+			(project "ScaleController_RevA"
 				(path "/16c571a0-8550-4f05-972c-22b0701cbf02/1a7f1cfb-b266-4842-99c6-585192ff3edb"
 					(reference "NT3")
@@
 		)
 		(instances
-			(project ""
+			(project "ScaleController_RevA"
 				(path "/16c571a0-8550-4f05-972c-22b0701cbf02/1a7f1cfb-b266-4842-99c6-585192ff3edb"
 					(reference "C17")
@@
 		)
 		(instances
-			(project ""
+			(project "ScaleController_RevA"
 				(path "/16c571a0-8550-4f05-972c-22b0701cbf02/1a7f1cfb-b266-4842-99c6-585192ff3edb"
 					(reference "#FLG03")
@@
 		)
 		(instances
-			(project ""
+			(project "ScaleController_RevA"
 				(path "/16c571a0-8550-4f05-972c-22b0701cbf02/1a7f1cfb-b266-4842-99c6-585192ff3edb"
 					(reference "C12")
@@
 			)
 		)
-		(property "Value" "+3.3V"
+		(property "Value" "3.3V"
 			(at 58.42 68.5799 90)
 			(effects
@@
 		)
 		(instances
-			(project ""
+			(project "ScaleController_RevA"
 				(path "/16c571a0-8550-4f05-972c-22b0701cbf02/1a7f1cfb-b266-4842-99c6-585192ff3edb"
 					(reference "#PWR031")
@@
 		)
 		(instances
-			(project ""
+			(project "ScaleController_RevA"
 				(path "/16c571a0-8550-4f05-972c-22b0701cbf02/1a7f1cfb-b266-4842-99c6-585192ff3edb"
 					(reference "#PWR035")
@@
 			)
 		)
-		(property "Value" "+3.3V"
+		(property "Value" "3.3V"
 			(at 160.02 54.6099 90)
 			(effects
@@
 		)
 		(instances
-			(project ""
+			(project "ScaleController_RevA"
 				(path "/16c571a0-8550-4f05-972c-22b0701cbf02/1a7f1cfb-b266-4842-99c6-585192ff3edb"
 					(reference "#PWR036")
@@
 		)
 		(instances
-			(project ""
+			(project "ScaleController_RevA"
 				(path "/16c571a0-8550-4f05-972c-22b0701cbf02/1a7f1cfb-b266-4842-99c6-585192ff3edb"
 					(reference "C16")
@@
 		)
 		(instances
-			(project ""
+			(project "ScaleController_RevA"
 				(path "/16c571a0-8550-4f05-972c-22b0701cbf02/1a7f1cfb-b266-4842-99c6-585192ff3edb"
 					(reference "C14")
@@
 		)
 		(instances
-			(project ""
+			(project "ScaleController_RevA"
 				(path "/16c571a0-8550-4f05-972c-22b0701cbf02/1a7f1cfb-b266-4842-99c6-585192ff3edb"
 					(reference "NT1")
@@
 		)
 		(instances
-			(project ""
+			(project "ScaleController_RevA"
 				(path "/16c571a0-8550-4f05-972c-22b0701cbf02/1a7f1cfb-b266-4842-99c6-585192ff3edb"
 					(reference "#PWR032")
@@
 		)
 		(instances
-			(project ""
+			(project "ScaleController_RevA"
 				(path "/16c571a0-8550-4f05-972c-22b0701cbf02/1a7f1cfb-b266-4842-99c6-585192ff3edb"
 					(reference "#PWR030")

Commit message: Fix HX711 input filter topology; remove stale test points
C12/C13 were in series with the load-cell signal (S -> 100R -> 4.7nF ->
INA), which blocks the DC bridge output. R15/R16 now feed INA+/INA-
directly and C12/C13 shunt those nodes to AGND. Removed TP2 (DOUT) and
TP4 (PD_SCK), leftovers from the KLP-5e board. Netlist: 64 nets, ERC 0
errors. PCB updated from schematic; 66 unrouted, DRC unchanged.

Co-Authored-By: Claude Fable 5.1 <noreply@anthropic.com>
Connections:
- net A+: now also R15.1
- net A-: now also R16.1
- net AGND: now also C12.1, C13.2
Changed lines of the file:
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@@
+	)
+	(junction
+		(at 52.07 77.47)
+		(diameter 0)
+		(color 0 0 0 0)
+	)
+	(junction
+		(at 52.07 87.63)
+		(diameter 0)
+		(color 0 0 0 0)
 	)
 	(junction
@@
 	(wire
 		(pts
-			(xy 52.07 96.52) (xy 52.07 81.28)
+			(xy 52.07 96.52) (xy 52.07 87.63)
 		)
 		(stroke
@@
 	(wire
 		(pts
-			(xy 44.45 68.58) (xy 44.45 77.47)
-		)
-		(stroke
-			(width 0)
-			(type default)
-		)
-	)
-	(wire
-		(pts
 			(xy 185.42 57.15) (xy 194.31 57.15)
 		)
@@
 	(wire
 		(pts
-			(xy 52.07 68.58) (xy 52.07 78.74)
+			(xy 44.45 87.63) (xy 52.07 87.63)
+		)
+		(stroke
+			(width 0)
+			(type default)
+		)
+	)
+	(wire
+		(pts
+			(xy 52.07 68.58) (xy 52.07 77.47)
 		)
 		(stroke
@@
 	(wire
 		(pts
+			(xy 44.45 77.47) (xy 52.07 77.47)
+		)
+		(stroke
+			(width 0)
+			(type default)
+		)
+	)
+	(wire
+		(pts
 			(xy 77.47 48.26) (xy 87.63 48.26)
 		)
@@
 	(wire
 		(pts
+			(xy 52.07 87.63) (xy 52.07 81.28)
+		)
+		(stroke
+			(width 0)
+			(type default)
+		)
+	)
+	(wire
+		(pts
 			(xy 184.15 72.39) (xy 194.31 72.39)
 		)
@@
 	(wire
 		(pts
+			(xy 41.91 68.58) (xy 44.45 68.58)
+		)
+		(stroke
+			(width 0)
+			(type default)
+		)
+	)
+	(wire
+		(pts
 			(xy 116.84 55.88) (xy 116.84 50.8)
 		)
@@
 	(wire
 		(pts
+			(xy 52.07 77.47) (xy 52.07 78.74)
+		)
+		(stroke
+			(width 0)
+			(type default)
+		)
+	)
+	(wire
+		(pts
 			(xy 62.23 62.23) (xy 66.04 62.23)
 		)
@@
 		(pts
 			(xy 100.33 52.07) (xy 100.33 55.88)
-		)
-		(stroke
-			(width 0)
-			(type default)
-		)
-	)
-	(wire
-		(pts
-			(xy 44.45 87.63) (xy 44.45 96.52)
 		)
 		(stroke
@@
 		)
 	)
+	(label "AGND"
+		(at 41.91 68.58 0)
+		(effects
+			(font
+				(size 1.27 1.27)
+			)
+			(justify left bottom)
+		)
+	)
 	(label "E-"
 		(at 185.42 88.9 180)
@@
 		(effects
 			(font
+				(size 1.27 1.27)
+			)
+			(justify right bottom)
+		)
+	)
+	(label "AGND"
+		(at 44.45 96.52 180)
+		(effects
+			(font

Commit message: Load-cell connectors: JST PH friction-lock, cells 3/4 inverted on-board
Schematic: J3/J5/J7/J8 footprints changed to JST_PH_B3B-PH-K_1x03 (top
entry, 2.0 mm, friction lock) replacing the plain Samtec MTMM pin
headers that would let plugs walk off. Connector symbol pins renumbered
01/02/03 -> 1/2/3 to match the JST pad numbering. One connector pair
(J3/J7 vs J5/J8) now has E+/E- swapped so all four half-bridge cells plug
in identically and the PCB provides the required inversion; the user no
longer swaps white/black on two cells. Note: as wired, the net named E+
ties to GND (NT3) and E- to 3.3V (NT2); functionally correct, naming to
tidy later.

Board: JST pads netted; rows spread to 5.7 mm pitch for the 5.5 mm
housings (column shifted 0.3 mm left to clear the cap column); NT2/NT3
moved above the connector column; excitation chains rebuilt with the
F.Cu/B.Cu crossover between rows 2 and 3; S+/S- links regenerated;
connector reference text hidden pending real silkscreen labels.
Verified on a fill-stripped copy: 0 violations, 0 unrouted. Fills stale
in this commit; refill in GUI.

Co-Authored-By: Claude Fable 5.1 <noreply@anthropic.com>
Parts:
- J3, J5, J7, J8: footprint MTMM-103-03-T-S-150:SAMTEC_MTMM-103-03-T-S-150 -> Connector_JST:JST_PH_B3B-PH-K_1x03_P2.00mm_Vertical
Connections:
- net E+: now also J3.3, J5.1, J7.3, J8.1, NT3.2; no longer J3.01, J5.01, J7.01, J8.01, NT2.2
- net E-: now also J3.1, J5.3, J7.1, J8.3, NT2.2; no longer J3.03, J5.03, J7.03, J8.03, NT3.2
- net S_MINUS_GRP: now also J5.2, J8.2; no longer J5.02, J8.02
- net S_PLUS_GRP: now also J3.2, J7.2; no longer J3.02, J7.02

Commit message: Swap E+/E- labels so E+ is the 3.3V-side excitation again
Pure rename: the four E+ and four E- labels on the HX711 sheet exchanged,
and the two net names on the board exchanged to match. No wire, pad or
track changed. Netlist: E+ = J3.1 J5.3 J7.1 J8.3 NT2.2 (3.3V tie);
E- = J3.3 J5.1 J7.3 J8.1 NT3.2 (GND tie). ERC 0 errors; DRC 0 unrouted,
4 warnings; every pad net on the board matches the schematic.

Co-Authored-By: Claude Fable 5.1 <noreply@anthropic.com>
Connections:
- net E+: now also J3.1, J5.3, J7.1, J8.3, NT2.2; no longer J3.3, J5.1, J7.3, J8.1, NT3.2
- net E-: now also J3.3, J5.1, J7.3, J8.1, NT3.2; no longer J3.1, J5.3, J7.1, J8.3, NT2.2
Changed lines of the file:
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@@
 		)
 	)
-	(label "E+"
+	(label "E-"
 		(at 185.42 59.69 180)
 		(effects
@@
 		)
 	)
-	(label "E-"
+	(label "E+"
 		(at 184.15 74.93 180)
 		(effects
@@
 		)
 	)
-	(label "E+"
+	(label "E-"
 		(at 185.42 97.79 180)
 		(effects
@@
 		)
 	)
-	(label "E-"
+	(label "E+"
 		(at 184.15 54.61 180)
 		(effects
@@
 		)
 	)
-	(label "E+"
+	(label "E-"
 		(at 184.15 69.85 180)
 		(effects
@@
 		)
 	)
-	(label "E-"
+	(label "E+"
 		(at 185.42 83.82 180)
 		(effects
@@
 		)
 	)
-	(label "E+"
+	(label "E-"
 		(at 185.42 88.9 180)
 		(effects
@@
 		)
 	)
-	(label "E-"
+	(label "E+"
 		(at 185.42 102.87 180)
 		(effects

Commit message: Pre-order tidy: DRU, symbol-lib sync, PCBWay stackup, JST part number on J3/5/7/8
- .kicad_dru: drop the global annular_width ignore. U3's ground-grid pads
  are 0.6/0.3 mm since the DFM pass; DRC is identical without the rule.
- Project symbol libs for LM1117MPX-3.3_NOPB, ESP32-C3-WROOM-02-H4 and
  MTMM-103-03-T-S-150 rewritten in KiCad 9 format from the schematic
  copies (the MTMM copy has pins 1/2/3 to match the JST PH pads; the old
  lib still had 01/02/03). SnapEDA "Description_1" junk fields removed
  from libs, embedded copies and instances. ERC: 0 lib_symbol_mismatch.
- Stackup: PCBWay standard 4-layer 1.6 mm (7628 prepreg 0.19 x2,
  core 1.03, 1 oz all layers).
- J3/J5/J7/J8: Value/MF/MP -> JST B3B-PH-K-S in schematic, project lib
  and board footprints; stale Samtec/SnapEDA fields dropped. Symbol name
  and lib_id left as MTMM-103-03-T-S-150.

Netlist nets/pins identical before and after. DRC with schematic parity:
0 errors, 0 unconnected, 0 parity issues, 5 known benign warnings.

Co-Authored-By: Claude Fable 5.1 <noreply@anthropic.com>
Parts:
- J3, J5, J7, J8: value MTMM-103-03-T-S-150 -> B3B-PH-K-S; Availability In Stock -> (none); Check_prices https://www.snapeda.com/parts/MTMM-103-03-T-S-150/Samtec/vi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 -> (none); Description_1 Connector Header Through Hole 3 position 0.079 (2.00mm) -> (none); MANUFACTURER SAMTEC -> JST; MF Samtec -> JST; MP MTMM-103-03-T-S-150 -> B3B-PH-K-S; Package None -> (none); Price None -> (none); SnapEDA_Link https://www.snapeda.com/parts/MTMM-103-03-T-S-150/Samtec/vi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 -> (none)

Commit message: BOM fixes, DRC exclusions, edge-clearance restore, fab outputs and order notes
- C9 value 4.7u -> 10u (matches its KEMET T491A 10 uF part number; LM1117
  output cap). Capacitor values normalised to 0.1u / 1u / 10u so identical
  0805 parts group: BOM 30 -> 27 lines.
- J1 value -> HRO TYPE-C-31-M-12, MF/MP fields added (schematic + board).
- min_copper_edge_clearance restored to 0.3 mm. The DFM commit 4617449 set
  it; the GUI refill save in 61ca090 wrote the old project file back (0.2).
  Board meets 0.3 (probe rule: no violations).
- DRC exclusions for the 4 silk-over-edge warnings (J1 face, U3 antenna
  notch), added in the GUI.
- docs/pcbway-order-notes.md: board spec, stackup, drills, special notes.
- docs/status-2026-09-18.md: supersedes 17 Sept; kicad-cli regen commands.
- TODO: fabrication items ticked.

Fab package generated to fabrication/RevA-2026-09-18/ (git-ignored):
schematic PDF, BOM (raw + PCBWay), Gerbers/drill zip, pos top/bottom.
Netlist nets/pins identical to bdae270. DRC + parity: 0 errors,
0 unconnected, 0 parity; 4 excluded + 1 intentional warning.

Co-Authored-By: Claude Fable 5.1 <noreply@anthropic.com>
Parts:
- C14: value 1 µF -> 1u
- C15, C17: value 0.1 µF -> 0.1u
- C16: value 10 µF -> 10u
Changed lines of the file:
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@@
 			)
 		)
-		(property "Value" "0.1 µF"
+		(property "Value" "0.1u"
 			(at 104.14 49.5299 0)
 			(effects
@@
 			)
 		)
-		(property "Value" "0.1 µF"
+		(property "Value" "0.1u"
 			(at 67.31 99.568 90)
 			(effects
@@
 			)
 		)
-		(property "Value" "10 µF"
+		(property "Value" "10u"
 			(at 120.65 48.2599 0)
 			(effects
@@
 			)
 		)
-		(property "Value" "1 µF"
+		(property "Value" "1u"
 			(at 69.85 57.15 90)
 			(effects

Commit message: Specify dielectric and source for the HX711 front-end parts in the BOM
- C12/C13: Value "4.7nF C0G 50V", description marks them as the matched
  HX711 input-filter pair, no Class 2 substitution.
- C16: Value "10u X7R 10V", description forbids Y5V.
- U6: MF/MP Avia Semiconductor HX711 added; description notes it is
  noise-critical and must be genuine or a known-good source.
- Order notes and status note updated accordingly.

Value fields are on F.Fab only; Gerbers unchanged. Netlist nets/pins
identical. DRC + parity: 0 errors, 0 parity issues.

Co-Authored-By: Claude Fable 5.1 <noreply@anthropic.com>
Parts:
- C12, C13: value 4.7nF -> 4.7nF C0G 50V
- C16: value 10u -> 10u X7R 10V
- U6: MF (none) -> Avia Semiconductor; MP (none) -> HX711
Changed lines of the file:
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@@
 			)
 		)
-		(property "Description" "24-bit Analog-to-Digital Converter (ADC) for Weight Scales, SOIC-16 (SOP-16)"
+		(property "MF" "Avia Semiconductor"
+			(at 93.98 80.01 0)
+			(effects
+				(font
+					(size 1.27 1.27)
+				)
+				(hide yes)
+			)
+		)
+		(property "MP" "HX711"
+			(at 93.98 80.01 0)
+			(effects
+				(font
+					(size 1.27 1.27)
+				)
+				(hide yes)
+			)
+		)
+		(property "Description" "24-bit ADC for weight scales, SOIC-16 - Avia Semiconductor HX711, genuine or known-good source (noise-critical)"
 			(at 90.17 78.74 0)
 			(effects
@@
 			)
 		)
-		(property "Value" "4.7nF"
+		(property "Value" "4.7nF C0G 50V"
 			(at 48.006 102.616 90)
 			(effects
@@
 			)
 		)
-		(property "Description" "Unpolarized capacitor"
+		(property "Description" "4.7 nF C0G/NP0 50 V, 0805 - HX711 input filter, matched pair with C12; do not substitute Class 2 dielectric"
 			(at 48.26 96.52 0)
 			(effects
@@
 			)
 		)
-		(property "Value" "4.7nF"
+		(property "Value" "4.7nF C0G 50V"
 			(at 48.26 63.5 90)
 			(effects
@@
 			)
 		)
-		(property "Description" "Unpolarized capacitor"
+		(property "Description" "4.7 nF C0G/NP0 50 V, 0805 - HX711 input filter, matched pair with C13; do not substitute Class 2 dielectric"
 			(at 48.26 68.58 0)
 			(effects
@@
 			)
 		)
-		(property "Value" "10u"
+		(property "Value" "10u X7R 10V"
 			(at 120.65 48.2599 0)
 			(effects
@@
 			)
 		)
-		(property "Description" "Unpolarized capacitor"
+		(property "Description" "10 uF X7R or X5R, 10 V min, 0805 - HX711 AVDD/DVDD decoupling; no Y5V"
 			(at 116.84 46.99 0)
 			(effects

Commit message: Schematic: title blocks (Scale Controller, rev A, 2026-09-18, per-sheet comments); replace stale CP2102 and ESP32-S3 notes
Co-Authored-By: Claude Fable 5.1 <noreply@anthropic.com>
Other:
- company: (none) -> Steve Maegley
- title: ESP32 sensor board -> Scale Controller
Changed lines of the file:
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@@
 	(paper "A4")
 	(title_block
-		(title "ESP32 sensor board")
-		(rev "1")
-		(comment 1 "OLED Header")
+		(title "Scale Controller")
+		(date "2026-09-18")
+		(rev "A")
+		(company "Steve Maegley")
+		(comment 1 "HX711 and load-cell sockets")
 	)
 	(rectangle
